File: PCB/namii65.kicad_pcb (KiCad board)
At the start: 2 copper layers, 304.8 x 95.2 mm, 146 parts, among them SW1 Esc, SW10 9, SW11 0, SW12 -_, SW13 =+, SW14 Backspace, SW15 Home, SW16 Tab, SW17 q, SW18 w, SW19 e, SW2 1, SW20 r, SW21 t, SW22 y, SW23 u, SW24 i, SW25 o, SW26 p, SW27 [ {, SW28 } ], SW29 \ |, SW3 2, SW30 End, SW31 Capslock, SW32 a, SW33 s, SW34 d, SW35 f, SW36 g, SW37 h, SW38 j, SW39 k, SW4 3, SW40 l, SW41 ; :, SW42 ' ", SW43 Enter, SW44 pg up, SW45 L shift, SW46 z, SW47 x, SW48 c, SW49 v, SW5 4, SW50 b, SW51 n, SW52 m, SW53 , <, SW54 . >, SW55 / ?, SW56 R shift, SW57 UP, SW58 pg down, SW59 L ctrl, SW6 5, SW60 L win, SW61 L alt, SW62 6,25u, SW63 R alt, SW64 R ctrl, SW65 LEFT, SW66 DOWN, SW67 RIGHT, SW68 L ctrl, SW69 L win, SW7 6, SW70 L ctrl, SW71 7u, SW72 R ctrl, SW8 7, SW9 8, U1 ProMicro

Commit message: adding production file
Parts:
- added H1: Logo, fikoz_lib:FIKOZ_logo_1, B.Cu at (195.8, 112.9)
- added SW73: Capslock, PCM_Switch_Keyboard_Hotswap_Kailh:SW_Hotswap_Kailh_MX_1.25u, F.Cu at (40.5, 76.2)
- moved D31 5.05 mm to (57.6, 79.9)
- turned SW31 to 180 degrees
Connections:
- SW31 pad 1: Col0 -> Net-(D31-A)
- SW31 pad 2: Net-(D31-A) -> Col0
Routing:
- net Net-(D31-A): track 7.58 -> 21.5 mm
- net Row4: track 226.2 -> 221.2 mm
- net Row7: track 434.8 -> 435.6 mm
- net Col0: track 268.2 -> 268.9 mm, vias 8 -> 9
- net Col2: track 331.4 -> 330.8 mm
- net Col3: track 273.7 -> 274.2 mm
