File: PCB/namii65.kicad_sch (KiCad schematic)
At the start: 146 parts, among them SW1 Esc, SW10 9, SW11 0, SW12 -_, SW13 =+, SW14 Backspace, SW15 Home, SW16 Tab, SW17 q, SW18 w, SW19 e, SW2 1, SW20 r, SW21 t, SW22 y, SW23 u, SW24 i, SW25 o, SW26 p, SW27 [ {, SW28 } ], SW29 \ |, SW3 2, SW30 End, SW31 Capslock, SW32 a, SW33 s, SW34 d, SW35 f, SW36 g, SW37 h, SW38 j, SW39 k, SW4 3, SW40 l, SW41 ; :, SW42 ' ", SW43 Enter, SW44 pg up, SW45 L shift, SW46 z, SW47 x, SW48 c, SW49 v, SW5 4, SW50 b, SW51 n, SW52 m, SW53 , <, SW54 . >, SW55 / ?, SW56 R shift, SW57 UP, SW58 pg down, SW59 L ctrl, SW6 5, SW60 L win, SW61 L alt, SW62 6,25u, SW63 R alt, SW64 R ctrl, SW65 LEFT, SW66 DOWN, SW67 RIGHT, SW68 L ctrl, SW69 L win, SW7 6, SW70 L ctrl, SW71 7u, SW72 R ctrl, SW8 7, SW9 8, U1 ProMicro

Commit message: adding production file
Parts:
- added H1: Logo, fikoz_lib:FIKOZ_logo_1, symbol keebio:Hole
- added SW73: Capslock, PCM_Switch_Keyboard_Hotswap_Kailh:SW_Hotswap_Kailh_MX_1.25u, symbol keebio:MX_LED
Connections:
- net Col0: now also SW31.2, SW73.1; no longer SW31.1
- net at D31.2 (A): now also SW31.1, SW73.2; no longer SW31.2
Changed lines of the file:
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@@
 	)
 	(junction
-		(at 63.5 194.31)
-		(diameter 0)
-		(color 0 0 0 0)
-	)
-	(junction
 		(at 86.36 194.31)
 		(diameter 0)
@@
 	)
 	(junction
+		(at 63.5 186.69)
+		(diameter 0)
+		(color 0 0 0 0)
+	)
+	(junction
 		(at 137.16 121.92)
 		(diameter 0)
@@
 	)
 	(junction
+		(at 63.5 194.31)
+		(diameter 0)
+		(color 0 0 0 0)
+	)
+	(junction
 		(at 63.5 242.57)
 		(diameter 0)
@@
 	)
 	(junction
+		(at 53.34 194.31)
+		(diameter 0)
+		(color 0 0 0 0)
+	)
+	(junction
 		(at 137.16 138.43)
 		(diameter 0)
@@
 	(polyline
 		(pts
-			(xy 146.05 43.18) (xy 193.675 43.18)
+			(xy 146.05 43.18) (xy 193.548 43.18)
 		)
 		(stroke
@@
 	(wire
 		(pts
-			(xy 63.5 156.21) (xy 63.5 194.31)
-		)
-		(stroke
-			(width 0)
-			(type default)
-		)
-	)
-	(wire
-		(pts
 			(xy 97.79 201.93) (xy 118.11 201.93)
 		)
@@
 	(wire
 		(pts
+			(xy 53.34 186.69) (xy 53.34 194.31)
+		)
+		(stroke
+			(width 0)
+			(type default)
+		)
+	)
+	(wire
+		(pts
 			(xy 160.02 138.43) (xy 181.61 138.43)
 		)
@@
 	(polyline
 		(pts
-			(xy 193.675 43.18) (xy 193.675 95.25)
+			(xy 193.548 43.18) (xy 193.675 95.25)
 		)
 		(stroke
@@
 	(wire
 		(pts
+			(xy 63.5 194.31) (xy 63.5 212.09)
+		)
+		(stroke
+			(width 0)
+			(type default)
+		)
+	)
+	(wire
+		(pts
 			(xy 222.25 138.43) (xy 245.11 138.43)
 		)
@@
 	(wire
 		(pts
-			(xy 63.5 194.31) (xy 63.5 212.09)
+			(xy 63.5 186.69) (xy 63.5 194.31)
 		)
 		(stroke
@@
 	(wire
 		(pts
+			(xy 63.5 156.21) (xy 63.5 186.69)
+		)
+		(stroke
+			(width 0)
+			(type default)
+		)
+	)
+	(wire
+		(pts
 			(xy 137.16 238.76) (xy 160.02 238.76)
 		)
@@
 		(lib_id "keebio:MX_LED")
 		(at 58.42 194.31 0)
-		(mirror y)
+		(mirror x)
 		(unit 1)
 		(exclude_from_sim no)
@@
 		(dnp no)
 		(property "Reference" "SW31"
-			(at 58.42 189.23 0)
+			(at 58.42 199.39 0)
 			(effects
 				(font
@@
 		)
 		(property "Value" "Capslock"
-			(at 58.42 187.96 0)
+			(at 58.42 200.66 0)
 			(effects
 				(font
@@
 	)
 	(symbol
+		(lib_id "keebio:Hole")
+		(at 160.02 54.61 0)
+		(unit 1)
+		(exclude_from_sim no)
+		(in_bom yes)
+		(on_board yes)
+		(dnp no)
+		(fields_autoplaced yes)
+		(property "Reference" "H1"
+			(at 165.1 53.3399 0)
+			(effects
+				(font
+					(size 1.524 1.524)
+				)
+				(justify left)
+			)
+		)
+		(property "Value" "Logo"
+			(at 165.1 55.8799 0)
+			(effects
+				(font
+					(size 1.524 1.524)
+				)
+				(justify left)
+			)
+		)
+		(property "Footprint" "fikoz_lib:FIKOZ_logo_1"
+			(at 160.02 54.61 0)
+			(effects
+				(font
+					(size 1.524 1.524)
+				)
+				(hide yes)
+			)
+		)
+		(property "Datasheet" ""
+			(at 160.02 54.61 0)
+			(effects
+				(font
+					(size 1.524 1.524)
+				)
+				(hide yes)
+			)
+		)
+		(property "Description" ""
+			(at 160.02 54.61 0)
+			(effects
+				(font
+					(size 1.27 1.27)
+				)
+				(hide yes)
+			)
+		)
+		(instances
+			(project ""
+				(path "/76079431-35ed-4353-aa72-18fd51045bd3"
+					(reference "H1")
+					(unit 1)
+				)
+			)
+		)
+	)
+	(symbol
 		(lib_id "Diode:1N4148W")
 		(at 201.93 255.27 90)
@@
 					(unit 1)
 				)
+			)
+		)
+	)
+	(symbol
+		(lib_id "keebio:MX_LED")
+		(at 58.42 186.69 0)
+		(mirror y)
+		(unit 1)
+		(exclude_from_sim no)
+		(in_bom yes)
+		(on_board yes)
+		(dnp no)
+		(property "Reference" "SW73"
+			(at 58.42 181.61 0)
+			(effects
+				(font
+					(size 1.27 1.27)
+				)
+				(hide yes)
+			)
+		)
+		(property "Value" "Capslock"
+			(at 58.42 180.34 0)
+			(effects
+				(font
+					(size 1.27 1.27)
+				)
+			)
+		)
+		(property "Footprint" "PCM_Switch_Keyboard_Hotswap_Kailh:SW_Hotswap_Kailh_MX_1.25u"
+			(at 58.42 186.69 0)
+			(effects
+				(font
+					(size 1.27 1.27)
+				)
+				(hide yes)
+			)
+		)
+		(property "Datasheet" ""
+			(at 58.42 186.69 0)
+			(effects
+				(font
+					(size 1.27 1.27)
+				)
+				(hide yes)
+			)
+		)
+		(property "Description" ""
+			(at 58.42 186.69 0)
+			(effects
+				(font
+					(size 1.27 1.27)
+				)
+				(hide yes)
+			)
+		)
+		(pin "1"
+		)
+		(pin "2"
+		)
+		(pin "3"
+		)
+		(pin "4"
+		)
+		(instances
+			(project "namii65"
+				(path "/76079431-35ed-4353-aa72-18fd51045bd3"
+					(reference "SW73")
+					(unit 1)
+				)
